File: nerve_ada_board.kicad_sch (KiCad schematic)
At the start: 64 parts, among them J10 CAN1, J11 CAN2, J2 TC2050-IDC, J3 2171750001, J5 WS2812B, J6 Camera, J7 PC12, PA4-7, J8 PC1-3, J9 PB4-5, SW1 SPST, SW2 SPST, SW3 SPST, U1 LD1117S33TR_SOT223, U2 STM32F446RET, U3 SAM-M10Q, U4 XBP9B-DMWT-002, U8 TXB0104QPWRQ1, U9 TXB0104QPWRQ1, Y1 8M, Y2 32k768

Commit message: Remove breakout GPIO PC12
Parts:
- removed J7: PC12, PA4-7, Connector_PinHeader_2.54mm:PinHeader_1x05_P2.54mm_Vertical, symbol Connector:Conn_01x05_Pin
- added J7: PA4-7, Connector_PinHeader_2.54mm:PinHeader_1x04_P2.54mm_Vertical, symbol Connector:Conn_01x04_Pin
Connections:
- net PA4: now also J7.1 (Pin_1)
- net PA5: now also J7.2 (Pin_2)
- net PA6: now also J7.3 (Pin_3)
- net PA7: now also J7.4 (Pin_4)
- net PC12: no longer names the net of U2.53 (PC12)
- no-connect marks 24 -> 25
Changed lines of the file:
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@@
 	)
 	(no_connect
+		(at 58.42 110.49)
+	)
+	(no_connect
 		(at 220.98 106.68)
 	)
@@
 	(wire
 		(pts
-			(xy 57.15 110.49) (xy 58.42 110.49)
-		)
-		(stroke
-			(width 0)
-			(type default)
-		)
-	)
-	(wire
-		(pts
 			(xy 60.96 187.96) (xy 62.23 187.96)
 		)
@@
 	(wire
 		(pts
-			(xy 21.59 153.67) (xy 22.86 153.67)
+			(xy 21.59 152.4) (xy 22.86 152.4)
 		)
 		(stroke
@@
 	(wire
 		(pts
-			(xy 21.59 156.21) (xy 22.86 156.21)
+			(xy 21.59 154.94) (xy 22.86 154.94)
 		)
 		(stroke
@@
 	(wire
 		(pts
-			(xy 21.59 161.29) (xy 22.86 161.29)
+			(xy 21.59 160.02) (xy 22.86 160.02)
 		)
 		(stroke
@@
 	(wire
 		(pts
-			(xy 21.59 158.75) (xy 22.86 158.75)
+			(xy 21.59 157.48) (xy 22.86 157.48)
 		)
 		(stroke
@@
 	(wire
 		(pts
-			(xy 21.59 151.13) (xy 22.86 151.13)
-		)
-		(stroke
-			(width 0)
-			(type default)
-		)
-	)
-	(wire
-		(pts
 			(xy 167.64 123.19) (xy 170.18 123.19)
 		)
@@
 		)
 	)
-	(text_box "GPIO"
-		(exclude_from_sim no)
-		(at 13.97 147.32 0)
-		(size 8.89 5.08)
-		(stroke
-			(width 0)
-			(type dash_dot_dot)
-		)
-		(fill
-			(type none)
-		)
-		(effects
-			(font
-				(size 1.27 1.27)
-				(thickness 0.254)
-				(bold yes)
-			)
-			(justify top)
-		)
-	)
 	(text_box "SPI"
 		(exclude_from_sim no)
-		(at 13.97 152.4 0)
+		(at 13.97 148.59 0)
 		(size 8.89 12.7)
 		(stroke
@@
 				(bold yes)
 			)
-			(justify bottom)
+			(justify top)
 		)
 	)
@@
 	(text "NO LEVEL SHIFT"
 		(exclude_from_sim no)
-		(at 29.21 152.654 0)
+		(at 28.956 152.654 0)
 		(effects
 			(font
@@
 	(hierarchical_label "PA5"
 		(shape input)
-		(at 21.59 156.21 180)
+		(at 21.59 154.94 180)
 		(fields_autoplaced yes)
 		(effects
@@
 		)
 	)
-	(hierarchical_label "PC12"
-		(shape input)
-		(at 21.59 151.13 180)
-		(fields_autoplaced yes)
-		(effects
-			(font
-				(size 1.27 1.27)
-			)
-			(justify right)
-		)
-	)
 	(hierarchical_label "SDIO_CMD"
 		(shape input)
@@
 	(hierarchical_label "PA7"
 		(shape input)
-		(at 21.59 161.29 180)
+		(at 21.59 160.02 180)
 		(fields_autoplaced yes)
 		(effects
@@
 		)
 	)
-	(hierarchical_label "PC12"
-		(shape input)
-		(at 57.15 110.49 180)
-		(fields_autoplaced yes)
-		(effects
-			(font
-				(size 1.27 1.27)
-			)
-			(justify right)
-		)
-	)
 	(hierarchical_label "CAN2_LOW-"
 		(shape input)
@@
 	(hierarchical_label "PA6"
 		(shape input)
-		(at 21.59 158.75 180)
+		(at 21.59 157.48 180)
 		(fields_autoplaced yes)
 		(effects
@@
 	(hierarchical_label "PA4"
 		(shape input)
-		(at 21.59 153.67 180)
+		(at 21.59 152.4 180)
 		(fields_autoplaced yes)
 		(effects
@@
 		(dnp no)
 		(fields_autoplaced yes)
-		(property "Reference" "#PWR054"
+		(property "Reference" "#PWR055"
 			(at 190.5 168.91 0)
 			(effects
@@
 			(project "nerve_ada_board"
 				(path "/c0277862-b3f2-4e0e-986f-34702f0543f0"
-					(reference "#PWR054")
+					(reference "#PWR055")
 					(unit 1)
 				)
@@
 		(on_board yes)
 		(dnp no)
-		(property "Reference" "#PWR049"
+		(property "Reference" "#PWR046"
 			(at 140.97 128.27 0)
 			(effects
@@
 			(project "nerve_ada_board"
 				(path "/c0277862-b3f2-4e0e-986f-34702f0543f0"
-					(reference "#PWR049")
+					(reference "#PWR046")
 					(unit 1)
 				)
@@
 		(dnp no)
 		(fields_autoplaced yes)
-		(property "Reference" "#PWR045"
+		(property "Reference" "#PWR047"
 			(at 185.42 130.81 0)
 			(effects
@@
 			(project "nerve_ada_board"
 				(path "/c0277862-b3f2-4e0e-986f-34702f0543f0"
-					(reference "#PWR045")
+					(reference "#PWR047")
 					(unit 1)
 				)
@@
 		(dnp no)
 		(fields_autoplaced yes)
-		(property "Reference" "#PWR047"
+		(property "Reference" "#PWR049"
 			(at 50.8 139.7 0)
 			(effects
@@
 			(project "nerve_ada_board"
 				(path "/c0277862-b3f2-4e0e-986f-34702f0543f0"
-					(reference "#PWR047")
+					(reference "#PWR049")
 					(unit 1)
 				)
@@
 	)
 	(symbol
+		(lib_id "Connector:Conn_01x04_Pin")
+		(at 27.94 154.94 0)
+		(mirror y)
+		(unit 1)
+		(exclude_from_sim no)
+		(in_bom yes)
+		(on_board yes)
+		(dnp no)
+		(property "Reference" "J7"
+			(at 28.956 154.686 0)
+			(effects
+				(font
+					(size 1.27 1.27)
+				)
+				(justify right)
+			)
+		)
+		(property "Value" "PA4-7"
+			(at 28.956 157.226 0)
+			(effects
+				(font
+					(size 1.27 1.27)
+				)
+				(justify right)
+			)
+		)
+		(property "Footprint" "Connector_PinHeader_2.54mm:PinHeader_1x04_P2.54mm_Vertical"
+			(at 27.94 154.94 0)
+			(effects
+				(font
+					(size 1.27 1.27)
+				)
+				(hide yes)
+			)
+		)
+		(property "Datasheet" "~"
+			(at 27.94 154.94 0)
+			(effects
+				(font
+					(size 1.27 1.27)
+				)
+				(hide yes)
+			)
+		)
+		(property "Description" "Generic connector, single row, 01x04, script generated"
+			(at 27.94 154.94 0)
+			(effects
+				(font
+					(size 1.27 1.27)
+				)
+				(hide yes)
+			)
+		)
+		(pin "2"
+		)
+		(pin "1"
+		)
+		(pin "4"
+		)
+		(pin "3"
+		)
+		(instances
+			(project "nerve_ada_board"
+				(path "/c0277862-b3f2-4e0e-986f-34702f0543f0"
+					(reference "J7")
+					(unit 1)
+				)
+			)
+		)
+	)
+	(symbol
 		(lib_id "Connector:Conn_01x03_Pin")
 		(at 203.2 66.04 0)
@@
 		(dnp no)
 		(fields_autoplaced yes)
-		(property "Reference" "#PWR046"
+		(property "Reference" "#PWR048"
 			(at 245.11 134.62 0)
 			(effects
@@
 			(project "nerve_ada_board"
 				(path "/c0277862-b3f2-4e0e-986f-34702f0543f0"
-					(reference "#PWR046")
+					(reference "#PWR048")
 					(unit 1)
 				)
@@
 	)
 	(symbol
-		(lib_id "Connector:Conn_01x05_Pin")
-		(at 27.94 156.21 0)
-		(mirror y)
-		(unit 1)
-		(exclude_from_sim no)
-		(in_bom yes)
-		(on_board yes)
-		(dnp no)
-		(fields_autoplaced yes)
-		(property "Reference" "J7"
-			(at 29.21 154.9399 0)
-			(effects
-				(font
-					(size 1.27 1.27)
-				)
-				(justify right)
-			)
-		)
-		(property "Value" "PC12, PA4-7"
-			(at 29.21 157.4799 0)
-			(effects
-				(font
-					(size 1.27 1.27)
-				)
-				(justify right)
-			)
-		)
-		(property "Footprint" "Connector_PinHeader_2.54mm:PinHeader_1x05_P2.54mm_Vertical"
-			(at 27.94 156.21 0)
-			(effects
-				(font
-					(size 1.27 1.27)
-				)
-				(hide yes)
-			)
-		)
-		(property "Datasheet" "~"
-			(at 27.94 156.21 0)
-			(effects
-				(font
-					(size 1.27 1.27)
-				)
-				(hide yes)
-			)
-		)
-		(property "Description" "Generic connector, single row, 01x05, script generated"
-			(at 27.94 156.21 0)
-			(effects
-				(font
-					(size 1.27 1.27)
-				)
-				(hide yes)
-			)
-		)
-		(pin "2"
-		)
-		(pin "3"
-		)
-		(pin "1"
-		)
-		(pin "4"
-		)
-		(pin "5"
-		)
-		(instances
-			(project ""
-				(path "/c0277862-b3f2-4e0e-986f-34702f0543f0"
-					(reference "J7")
-					(unit 1)
-				)
-			)
-		)
-	)
-	(symbol
 		(lib_id "power:GND")
 		(at 168.91 74.93 0)
@@
 		(on_board yes)
 		(dnp no)
-		(property "Reference" "#PWR048"
+		(property "Reference" "#PWR045"
 			(at 113.03 128.27 0)
 			(effects
@@
 			(project "nerve_ada_board"
 				(path "/c0277862-b3f2-4e0e-986f-34702f0543f0"
-					(reference "#PWR048")
+					(reference "#PWR045")
 					(unit 1)
 				)
@@
 		(dnp no)
 		(fields_autoplaced yes)
-		(property "Reference" "#PWR056"
+		(property "Reference" "#PWR054"
 			(at 143.51 158.75 0)
 			(effects
@@
 			(project "nerve_ada_board"
 				(path "/c0277862-b3f2-4e0e-986f-34702f0543f0"
-					(reference "#PWR056")
+					(reference "#PWR054")
 					(unit 1)
 				)
@@
 		(dnp no)
 		(fields_autoplaced yes)
-		(property "Reference" "#PWR055"
+		(property "Reference" "#PWR056"
 			(at 247.65 168.91 0)
 			(effects
@@
 			(project "nerve_ada_board"
 				(path "/c0277862-b3f2-4e0e-986f-34702f0543f0"
-					(reference "#PWR055")
+					(reference "#PWR056")
 					(unit 1)
 				)

Commit message: Update CR1220 battery holder component
Parts:
- removed BT1: CR1220, common:harwin_s8411-45r_cr1220_coin_battery_cell, symbol common:harwin_s8411-45r_cr1220_coin_battery_cell
- added BT1: CR1220, common:harwin_s8411-45r_cr1220, symbol common:harwin_s8411-45r_cr1220
Connections:
- net +3.3VBATT: now also BT1.2
- net GND: now also BT1.1
Changed lines of the file:
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@@
 	)
 	(symbol
-		(lib_id "common:harwin_s8411-45r_cr1220_coin_battery_cell")
-		(at 152.4 25.4 0)
-		(unit 1)
-		(exclude_from_sim no)
-		(in_bom yes)
-		(on_board yes)
-		(dnp no)
-		(property "Reference" "BT1"
-			(at 152.4 19.05 0)
-			(effects
-				(font
-					(size 1.27 1.27)
-				)
-			)
-		)
-		(property "Value" "CR1220"
-			(at 152.4 21.59 0)
-			(effects
-				(font
-					(size 1.27 1.27)
-				)
-			)
-		)
-		(property "Footprint" "common:harwin_s8411-45r_cr1220_coin_battery_cell"
-			(at 156.21 27.94 0)
-			(effects
-				(font
-					(size 1.27 1.27)
-				)
-				(hide yes)
-			)
-		)
-		(property "Datasheet" "https://www.harwin.com/products/S8411-45R"
-			(at 187.96 32.893 0)
-			(effects
-				(font
-					(size 1.27 1.27)
-				)
-				(hide yes)
-			)
-		)
-		(property "Description" "Battery Holder (Open) Coin, 12.0mm 1 Cell SMD (SMT) Tab"
-			(at 187.96 29.083 0)
-			(effects
-				(font
-					(size 1.27 1.27)
-				)
-				(hide yes)
-			)
-		)
-		(property "Manufacturer" "Harwin"
-			(at 187.96 24.003 0)
-			(effects
-				(font
-					(size 1.27 1.27)
-				)
-				(hide yes)
-			)
-		)
-		(property "Manufacturer Part Number" "S8411-45R"
-			(at 187.96 24.003 0)
-			(effects
-				(font
-					(size 1.27 1.27)
-				)
-				(hide yes)
-			)
-		)
-		(property "Distributor" "DigiKey"
-			(at 187.96 24.003 0)
-			(effects
-				(font
-					(size 1.27 1.27)
-				)
-				(hide yes)
-			)
-		)
-		(property "Distributor Part Number" "952-1745-1-ND"
-			(at 187.96 32.893 0)
-			(effects
-				(font
-					(size 1.27 1.27)
-				)
-				(hide yes)
-			)
-		)
-		(property "Distributor Link" "https://www.digikey.ca/en/products/detail/harwin-inc/S8411-45R/3131055?s=N4IgTCBcDaIMoA4AsBGFBaJBWASiAugL5A"
-			(at 187.96 29.083 0)
-			(effects
-				(font
-					(size 1.27 1.27)
-				)
-				(hide yes)
-			)
-		)
-		(pin "1"
-		)
-		(pin "2"
-		)
-		(instances
-			(project ""
-				(path "/c0277862-b3f2-4e0e-986f-34702f0543f0"
-					(reference "BT1")
-					(unit 1)
-				)
-			)
-		)
-	)
-	(symbol
 		(lib_id "power:+5V")
 		(at 152.4 57.15 0)
@@
 					(unit 1)
 				)
+			)
+		)
+	)
+	(symbol
+		(lib_id "common:harwin_s8411-45r_cr1220")
+		(at 152.4 25.4 0)
+		(unit 1)
+		(exclude_from_sim no)
+		(in_bom yes)
+		(on_board yes)
+		(dnp no)
+		(property "Reference" "BT1"
+			(at 152.4 19.05 0)
+			(effects
+				(font
+					(size 1.27 1.27)
+				)
+			)
+		)
+		(property "Value" "CR1220"
+			(at 152.4 21.59 0)
+			(effects
+				(font
+					(size 1.27 1.27)
+				)
+			)
+		)
+		(property "Footprint" "common:harwin_s8411-45r_cr1220"
+			(at 156.21 27.94 0)
+			(effects
+				(font
+					(size 1.27 1.27)
+				)
+				(hide yes)
+			)
+		)
+		(property "Datasheet" "https://www.harwin.com/products/S8411-45R"
+			(at 187.96 32.893 0)
+			(effects
+				(font
+					(size 1.27 1.27)
+				)
+				(hide yes)
+			)
+		)
+		(property "Description" "Battery Holder (Open) Coin, 12.0mm 1 Cell SMD (SMT) Tab"
+			(at 187.96 29.083 0)
+			(effects
+				(font
+					(size 1.27 1.27)
+				)
+				(hide yes)
+			)
+		)
+		(property "Manufacturer" "Harwin"
+			(at 187.96 24.003 0)
+			(effects
+				(font
+					(size 1.27 1.27)
+				)
+				(hide yes)
+			)
+		)
+		(property "Manufacturer Part Number" "S8411-45R"
+			(at 187.96 24.003 0)
+			(effects
+				(font
+					(size 1.27 1.27)
+				)
+				(hide yes)
+			)
+		)
+		(property "Distributor" "DigiKey"
+			(at 187.96 24.003 0)
+			(effects
+				(font
+					(size 1.27 1.27)
+				)
+				(hide yes)
+			)
+		)
+		(property "Distributor Part Number" "952-1745-1-ND"
+			(at 187.96 32.893 0)
+			(effects
+				(font
+					(size 1.27 1.27)
+				)
+				(hide yes)
+			)
+		)
+		(property "Distributor Link" "https://www.digikey.ca/en/products/detail/harwin-inc/S8411-45R/3131055?s=N4IgTCBcDaIMoA4AsBGFBaJBWASiAugL5A"
+			(at 187.96 29.083 0)
+			(effects
+				(font
+					(size 1.27 1.27)
+				)
+				(hide yes)
+			)
+		)
+		(pin "1"
+		)
+		(pin "2"
+		)
+		(instances
+			(project ""
+				(path "/c0277862-b3f2-4e0e-986f-34702f0543f0"
+					(reference "BT1")
+					(unit 1)
+				)

Commit message: Update CR1220 component, again
Parts:
- removed BT1: CR1220, common:harwin_s8411-45r_cr1220, symbol common:harwin_s8411-45r_cr1220
- added BT1: CR1220, common:harwin_s8411-45r_cr1220_battery, symbol common:harwin_s8411-45r_cr1220_battery
Connections:
- net +3.3VBATT: now also BT1.2
- net GND: now also BT1.1
Changed lines of the file:
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@@
+	)
+	(symbol
+		(lib_id "common:harwin_s8411-45r_cr1220_battery")
+		(at 152.4 25.4 0)
+		(unit 1)
+		(exclude_from_sim no)
+		(in_bom yes)
+		(on_board yes)
+		(dnp no)
+		(property "Reference" "BT1"
+			(at 152.4 19.05 0)
+			(effects
+				(font
+					(size 1.27 1.27)
+				)
+			)
+		)
+		(property "Value" "CR1220"
+			(at 152.4 21.59 0)
+			(effects
+				(font
+					(size 1.27 1.27)
+				)
+			)
+		)
+		(property "Footprint" "common:harwin_s8411-45r_cr1220_battery"
+			(at 156.21 27.94 0)
+			(effects
+				(font
+					(size 1.27 1.27)
+				)
+				(hide yes)
+			)
+		)
+		(property "Datasheet" "https://www.harwin.com/products/S8411-45R"
+			(at 187.96 32.893 0)
+			(effects
+				(font
+					(size 1.27 1.27)
+				)
+				(hide yes)
+			)
+		)
+		(property "Description" "Battery Holder (Open) Coin, 12.0mm 1 Cell SMD (SMT) Tab"
+			(at 187.96 29.083 0)
+			(effects
+				(font
+					(size 1.27 1.27)
+				)
+				(hide yes)
+			)
+		)
+		(property "Manufacturer" "Harwin"
+			(at 187.96 24.003 0)
+			(effects
+				(font
+					(size 1.27 1.27)
+				)
+				(hide yes)
+			)
+		)
+		(property "Manufacturer Part Number" "S8411-45R"
+			(at 187.96 24.003 0)
+			(effects
+				(font
+					(size 1.27 1.27)
+				)
+				(hide yes)
+			)
+		)
+		(property "Distributor" "DigiKey"
+			(at 187.96 24.003 0)
+			(effects
+				(font
+					(size 1.27 1.27)
+				)
+				(hide yes)
+			)
+		)
+		(property "Distributor Part Number" "952-1745-1-ND"
+			(at 187.96 32.893 0)
+			(effects
+				(font
+					(size 1.27 1.27)
+				)
+				(hide yes)
+			)
+		)
+		(property "Distributor Link" "https://www.digikey.ca/en/products/detail/harwin-inc/S8411-45R/3131055?s=N4IgTCBcDaIMoA4AsBGFBaJBWASiAugL5A"
+			(at 187.96 29.083 0)
+			(effects
+				(font
+					(size 1.27 1.27)
+				)
+				(hide yes)
+			)
+		)
+		(pin "1"
+		)
+		(pin "2"
+		)
+		(instances
+			(project ""
+				(path "/c0277862-b3f2-4e0e-986f-34702f0543f0"
+					(reference "BT1")
+					(unit 1)
+				)
+			)
+		)
 	)
 	(symbol
@@
 					(unit 1)
 				)
-			)
-		)
-	)
-	(symbol
-		(lib_id "common:harwin_s8411-45r_cr1220")
-		(at 152.4 25.4 0)
-		(unit 1)
-		(exclude_from_sim no)
-		(in_bom yes)
-		(on_board yes)
-		(dnp no)
-		(property "Reference" "BT1"
-			(at 152.4 19.05 0)
-			(effects
-				(font
-					(size 1.27 1.27)
-				)
-			)
-		)
-		(property "Value" "CR1220"
-			(at 152.4 21.59 0)
-			(effects
-				(font
-					(size 1.27 1.27)
-				)
-			)
-		)
-		(property "Footprint" "common:harwin_s8411-45r_cr1220"
-			(at 156.21 27.94 0)
-			(effects
-				(font
-					(size 1.27 1.27)
-				)
-				(hide yes)
-			)
-		)
-		(property "Datasheet" "https://www.harwin.com/products/S8411-45R"
-			(at 187.96 32.893 0)
-			(effects
-				(font
-					(size 1.27 1.27)
-				)
-				(hide yes)
-			)
-		)
-		(property "Description" "Battery Holder (Open) Coin, 12.0mm 1 Cell SMD (SMT) Tab"
-			(at 187.96 29.083 0)
-			(effects
-				(font
-					(size 1.27 1.27)
-				)
-				(hide yes)
-			)
-		)
-		(property "Manufacturer" "Harwin"
-			(at 187.96 24.003 0)
-			(effects
-				(font
-					(size 1.27 1.27)
-				)
-				(hide yes)
-			)
-		)
-		(property "Manufacturer Part Number" "S8411-45R"
-			(at 187.96 24.003 0)
-			(effects
-				(font
-					(size 1.27 1.27)
-				)
-				(hide yes)
-			)
-		)
-		(property "Distributor" "DigiKey"
-			(at 187.96 24.003 0)
-			(effects
-				(font
-					(size 1.27 1.27)
-				)
-				(hide yes)
-			)
-		)
-		(property "Distributor Part Number" "952-1745-1-ND"
-			(at 187.96 32.893 0)
-			(effects
-				(font
-					(size 1.27 1.27)
-				)
-				(hide yes)
-			)
-		)
-		(property "Distributor Link" "https://www.digikey.ca/en/products/detail/harwin-inc/S8411-45R/3131055?s=N4IgTCBcDaIMoA4AsBGFBaJBWASiAugL5A"
-			(at 187.96 29.083 0)
-			(effects
-				(font
-					(size 1.27 1.27)
-				)
-				(hide yes)
-			)
-		)
-		(pin "1"
-		)
-		(pin "2"
-		)
-		(instances
-			(project ""
-				(path "/c0277862-b3f2-4e0e-986f-34702f0543f0"
-					(reference "BT1")
-					(unit 1)
-				)
